Commit message: Correct SO101 workcell planning model

File: src/so101_moveit_config/description/so101_follower.urdf.xacro (robot description, xacro)
@@ -14,7 +14,18 @@
     <color rgba="0.91 0.86 0.74 1" />
   </material>
+  <material name="pgripper_hardware">
+    <color rgba="0.32 0.33 0.34 1" />
+  </material>
   <xacro:macro name="mesh_geometry" params="file">
     <geometry>
       <mesh filename="package://so101_moveit_config/description/assets/${file}" />
+    </geometry>
+  </xacro:macro>
+  <xacro:macro name="millimeter_mesh_geometry" params="file">
+    <geometry>
+      <mesh
+        filename="package://so101_moveit_config/description/assets/${file}"
+        scale="0.001 0.001 0.001"
+      />
     </geometry>
   </xacro:macro>
@@ -72,30 +83,30 @@
         name="Rotation_R"
         initial="0.0"
-        min_position="-1.6158680162694754"
-        max_position="1.6158680162694754"
+        min_position="-2.16"
+        max_position="2.16"
       />
       <xacro:controlled_joint
         name="Pitch_R"
         initial="1.575"
-        min_position="-0.21731888570186922"
-        max_position="3.367318885701869"
+        min_position="-0.24"
+        max_position="3.56"
       />
       <xacro:controlled_joint
         name="Elbow_R"
         initial="1.46"
-        min_position="-0.21800940941740532"
-        max_position="3.138009409417405"
+        min_position="-0.47"
+        max_position="3.40"
       />
       <xacro:controlled_joint
         name="Wrist_Pitch_R"
         initial="0.0"
-        min_position="-1.7317119080013874"
-        max_position="1.731711787879228"
+        min_position="-1.86"
+        max_position="1.94"
       />
       <xacro:controlled_joint
         name="Wrist_Roll_R"
         initial="1.5707963267948966"
-        min_position="-1.5533430342749532"
-        max_position="4.694935687864747"
+        min_position="-3.15"
+        max_position="3.15"
       />
       <xacro:controlled_joint
@@ -108,4 +119,48 @@
   </xacro:macro>
   <link name="world" />
+  <!--
+    Static bimanual workcell from the authoritative MuJoCo twin. Both arm
+    plates remain visible even though this config controls only the attached
+    right follower. The stand is visual-only, matching the source model.
+  -->
+  <link name="overhead_stand">
+    <visual name="stand_bottom">
+      <origin xyz="-0.0187 0.0365 0" rpy="1.5707963 0 0" />
+      <xacro:millimeter_mesh_geometry file="cam_mount_bottom.stl" />
+      <material name="galaxy_black" />
+    </visual>
+    <visual name="stand_middle">
+      <origin xyz="0 0 0.1885" rpy="1.5707963 0 0" />
+      <xacro:millimeter_mesh_geometry file="cam_mount_middle.stl" />
+      <material name="galaxy_black" />
+    </visual>
+    <visual name="stand_top">
+      <origin xyz="0 0 0.1885" rpy="1.5707963 0 0" />
+      <xacro:millimeter_mesh_geometry file="cam_mount_top.stl" />
+      <material name="galaxy_black" />
+    </visual>
+    <visual name="left_arm_plate">
+      <origin xyz="0.0753 0.0626 0.005" rpy="1.5707963 0 0" />
+      <xacro:millimeter_mesh_geometry file="arm_base.stl" />
+      <material name="galaxy_black" />
+    </visual>
+    <visual name="right_arm_plate">
+      <origin xyz="0.0753 -0.1695 0.005" rpy="1.5707963 0 0" />
+      <xacro:millimeter_mesh_geometry file="arm_base.stl" />
+      <material name="galaxy_black" />
+    </visual>
+    <visual name="overhead_cam_module">
+      <origin
+        xyz="0.07769 -0.00373 0.54222"
+        rpy="-1.1045436248526044 1.5510380297980149 0.4708007064179038"
+      />
+      <xacro:millimeter_mesh_geometry file="XLeRobot_camera2.stl" />
+      <material name="motor" />
+    </visual>
+  </link>
+  <joint name="world_to_overhead_stand" type="fixed">
+    <parent link="world" />
+    <child link="overhead_stand" />
+  </joint>
   <link name="Base_2">
     <inertial>
@@ -175,6 +230,6 @@
     <axis xyz="0 -1 0" />
     <limit
-      lower="-1.6158680162694754"
-      upper="1.6158680162694754"
+      lower="-2.16"
+      upper="2.16"
       effort="3.35"
       velocity="0.30"
@@ -216,6 +271,6 @@
     <axis xyz="-1 0 0" />
     <limit
-      lower="-0.21731888570186922"
-      upper="3.367318885701869"
+      lower="-0.24"
+      upper="3.56"
       effort="3.35"
       velocity="0.30"
@@ -257,6 +312,6 @@
     <axis xyz="1 0 0" />
     <limit
-      lower="-0.21800940941740532"
-      upper="3.138009409417405"
+      lower="-0.47"
+      upper="3.40"
       effort="3.35"
       velocity="0.30"
@@ -298,6 +353,6 @@
     <axis xyz="1 0 0" />
     <limit
-      lower="-1.7317119080013874"
-      upper="1.731711787879228"
+      lower="-1.86"
+      upper="1.94"
       effort="3.35"
       velocity="0.30"
@@ -320,18 +375,65 @@
     <visual>
       <origin xyz="0 -0.027975 -0.03525" rpy="0 0 -1.5707963267948966" />
-      <geometry>
-        <mesh
-          filename="package://so101_moveit_config/description/assets/norma_pgripper/gripper_base.stl"
-          scale="0.001 0.001 0.001"
-        />
-      </geometry>
-      <material name="cream_white" />
-    </visual>
-    <collision>
-      <origin xyz="0 -0.040 0" />
-      <geometry>
-        <box size="0.052 0.100 0.076" />
-      </geometry>
-    </collision>
+      <xacro:millimeter_mesh_geometry file="norma_pgripper/gripper_base.stl" />
+      <material name="cream_white" />
+    </visual>
+    <visual>
+      <origin
+        xyz="-0.02325 -0.023375 -0.01525"
+        rpy="0 0 1.5707963267948966"
+      />
+      <xacro:millimeter_mesh_geometry
+        file="norma_pgripper/gripper_base_shield.stl"
+      />
+      <material name="cream_white" />
+    </visual>
+    <visual>
+      <origin
+        xyz="0.023146893 -0.023375 0.01525"
+        rpy="3.141592653589793 0 1.5707963267948966"
+      />
+      <xacro:millimeter_mesh_geometry
+        file="norma_pgripper/gripper_base_shield.stl"
+      />
+      <material name="cream_white" />
+    </visual>
+    <visual>
+      <origin
+        xyz="0 -0.00925 -0.03275"
+        rpy="1.5707963267948966 0 3.141592653589793"
+      />
+      <xacro:millimeter_mesh_geometry
+        file="norma_pgripper/wiring_bracket.stl"
+      />
+      <material name="cream_white" />
+    </visual>
+    <visual>
+      <origin
+        xyz="0 -0.015785372 0.01525"
+        rpy="0 0 -1.5707963267948966"
+      />
+      <xacro:millimeter_mesh_geometry
+        file="norma_pgripper/camera_mount_square_27mm.stl"
+      />
+      <material name="cream_white" />
+    </visual>
+    <visual>
+      <xacro:millimeter_mesh_geometry
+        file="norma_pgripper/norma_st3215_servo.stl"
+      />
+      <material name="motor" />
+    </visual>
+    <visual>
+      <xacro:millimeter_mesh_geometry
+        file="norma_pgripper/norma_gripper_hardware.stl"
+      />
+      <material name="pgripper_hardware" />
+    </visual>
+    <visual>
+      <xacro:millimeter_mesh_geometry
+        file="norma_pgripper/norma_u20_camera.stl"
+      />
+      <material name="motor" />
+    </visual>
   </link>
   <joint name="Wrist_Roll_R" type="revolute">
@@ -341,6 +443,6 @@
     <axis xyz="0 -1 0" />
     <limit
-      lower="-1.5533430342749532"
-      upper="4.694935687864747"
+      lower="-3.15"
+      upper="3.15"
       effort="3.35"
       velocity="0.30"
@@ -431,5 +533,5 @@
     </inertial>
     <visual>
-      <origin rpy="0 0 1.5707963267948966" />
+      <origin rpy="1.5707963267948966 0 3.141592653589793" />
       <geometry>
         <mesh
